Commit message: HyQ is able to make a circle with only one foot

File: data/hyq/hyq.urdf (robot description, URDF)
Before this commit: robot plane, 13 links, 12 joints
Links:
- added link FL_EndEffector_point, mass 0.241
- added link FR_EndEffector_point, mass 0.241
- added link RL_EndEffector_point, mass 0.241
- added link RR_EndEffector_point, mass 0.241
- link chassis: geometry visual mesh filename=trunk/trunk.dae scale=1 1 1
Joints:
- added joint FL_EndEffector: type continuous, parent FL_lower_leg, child FL_EndEffector_point, origin xyz=0 -0.3 0.11 rpy=0 0 0, axis 1 0 0, limit effort=100 velocity=100
- added joint FR_EndEffector: type continuous, parent FR_lower_leg, child FR_EndEffector_point, origin xyz=0 -0.3 0.11 rpy=0 0 0, axis 1 0 0, limit effort=100 velocity=100
- added joint RL_EndEffector: type continuous, parent RL_lower_leg, child RL_EndEffector_point, origin xyz=0 -0.3 0.11 rpy=0 0 0, axis 1 0 0, limit effort=100 velocity=100
- added joint RR_EndEffector: type continuous, parent RR_lower_leg, child RR_EndEffector_point, origin xyz=0 -0.3 0.11 rpy=0 0 0, axis 1 0 0, limit effort=100 velocity=100

Commit message: hyq can make a circle for foot

File: data/hyq/hyq.urdf (robot description, URDF)
Before this commit: robot hyq, 17 links, 16 joints
Joints:
- joint FL_hip_motor_2_chassis_joint: origin xyz=0.15 0 0.242889 rpy=0 0 0 -> xyz=0.15 0 0.15 rpy=0 0 0
- joint FR_hip_motor_2_chassis_joint: origin xyz=-0.15 0 0.242889 rpy=0 0 0 -> xyz=-0.15 0 0.15 rpy=0 0 0
- joint RL_EndEffector: origin xyz=0 -0.3 0.11 rpy=0 0 0 -> xyz=0 -0.3 -0.11 rpy=0 0 0
- joint RR_EndEffector: origin xyz=0 -0.3 0.11 rpy=0 0 0 -> xyz=0 -0.3 -0.11 rpy=0 0 0
